File: recruiting.kicad_pcb (KiCad board)
At the start: 2 copper layers, 1 part

Commit message: Create PCB
Parts:
- added C2: 2u, Capacitor_THT:C_Axial_L3.8mm_D2.6mm_P7.50mm_Horizontal, F.Cu at (166.6, 69.8)
- added D1: LED, LED_SMD:LED_1206_3216Metric, F.Cu at (160.2, 76.1)
- added H1: MountingHole, MountingHole:MountingHole_2mm, F.Cu at (109.4, 78.7)
- added H2: MountingHole, MountingHole:MountingHole_2mm, F.Cu at (109.4, 95.2)
- added H3: MountingHole, MountingHole:MountingHole_2mm, F.Cu at (175.5, 78.7)
- added J1: Screw_Terminal_01x02, TerminalBlock_4Ucon:TerminalBlock_4Ucon_1x02_P3.50mm_Horizontal, F.Cu at (106.9, 68.6)
- added J2: Screw_Terminal_01x02, TerminalBlock_4Ucon:TerminalBlock_4Ucon_1x02_P3.50mm_Horizontal, F.Cu at (106.7, 101.6)
- added J3: Screw_Terminal_01x02, TerminalBlock_4Ucon:TerminalBlock_4Ucon_1x02_P3.50mm_Horizontal, F.Cu at (106.7, 85.1)
- added R1: 470, Resistor_SMD:R_1206_3216Metric, F.Cu at (164.0, 76.0)
- added R2: 7.5k, Resistor_SMD:R_1206_3216Metric, F.Cu at (115.8, 71.1)
- added R3: 500k, Resistor_SMD:R_1206_3216Metric, F.Cu at (143.7, 74.9)
- added R4: 1, Resistor_SMD:R_1206_3216Metric, F.Cu at (114.3, 76.2)
- added R5: 1k, Resistor_SMD:R_1206_3216Metric, F.Cu at (115.8, 68.6)
- added R6: 100k, Resistor_SMD:R_1206_3216Metric, F.Cu at (161.5, 69.8)
- added U1: ATA00F18S-L, Converter_DCDC:Converter_DCDC_Artesyn_ATA_SMD, F.Cu at (167.6, 94.0)
- added U2: JTD2048D05, Converter_DCDC:Converter_DCDC_XP_POWER_JTDxxxxxxx_THT, F.Cu at (144.8, 91.4)
- added U3: LM741, Package_DIP:DIP-8-16_W7.62mm, F.Cu at (120.7, 77.5)
- added U4: NE555P, Package_DIP:DIP-8_W7.62mm, F.Cu at (148.6, 77.5)
- C1: value 1F -> 100n; footprint Capacitor_SMD:C_0805_2012Metric -> Capacitor_SMD:CP_Elec_3x5.3
- moved C1 23.3 mm to (170.4, 76.2)
Connections:
- C1 pad 2: Net-(C1-Pad1) -> GND
Routing:
- net GND: track 0.00 -> 189.4 mm, vias 0 -> 2
- net +5V: track 0.00 -> 156.0 mm, vias 0 -> 1
- net /Vin_DCDC: track 0.00 -> 72.0 mm
- net Net-(R5-Pad2): track 0.00 -> 48.1 mm
- net Net-(C1-Pad1): track 57.5 -> 15.3 mm
- net Net-(R2-Pad2): track 0.00 -> 29.2 mm
- net Net-(C2-Pad1): track 0.00 -> 26.1 mm
- net /power_monitor/Over_10W: track 0.00 -> 23.5 mm
- net /Vout_3V3: track 0.00 -> 18.3 mm
- net /Vin_11-27: track 0.00 -> 13.6 mm
- net /power_monitor/LED_5V: track 0.00 -> 7.59 mm
- net Net-(D1-Pad1): track 0.00 -> 3.86 mm
Other:
- board outline added: 78.7 x 43.2 mm
- board text added: "+"
- board text added: "3V3"
- board text added: "5V"
