File: recruiting.kicad_sch (KiCad schematic)
At the start: 1 part

Commit message: Add project
Parts:
- removed C1: 1F, Capacitor_SMD:C_0805_2012Metric, symbol Device:C
- added J1: Morsetto 11-27V, Connector_Phoenix_MC_HighVoltage:PhoenixContact_MCV_1,5_2-G-5.08_1x02_P5.08mm_Vertical, symbol Connector:Screw_Terminal_01x02
- added J2: Morsetto 5V3A, Connector_Phoenix_MC_HighVoltage:PhoenixContact_MCV_1,5_2-G-5.08_1x02_P5.08mm_Vertical, symbol Connector:Screw_Terminal_01x02
- added J3: Morsetto 3,3V 0,5A, Connector_Phoenix_MC_HighVoltage:PhoenixContact_MCV_1,5_2-G-5.08_1x02_P5.08mm_Vertical, symbol Connector:Screw_Terminal_01x02
Connections:
- new net 3.3V0.5A: J3.1 (Pin_1)
- new net 5V3A: J2.1 (Pin_1)
- new net DC INPUT: J1.2 (Pin_2)
- new net GND: J1.1 (Pin_1), J2.2 (Pin_2), J3.2 (Pin_2)
Other:
- added sheet Alimentatore 3.3V (Alimentatore3V3.kicad_sch)
- added sheet Alimentatore 5V (Alimentatore5V.kicad_sch)
- added sheet Alimentatore 8V1 (Alimentatore8V.kicad_sch)
- added sheet Led control (Led_control.kicad_sch)
- added sheet Power meter (Power_meter.kicad_sch)
- title: Template -> Dc to Dc Step Down module
