File: pwr_monitor.kicad_sch (KiCad schematic)
At the start: 9 parts

Commit message: Create PCB
Parts:
- C1: renamed from C?; footprint (none) -> Capacitor_SMD:CP_Elec_3x5.3
- C2: renamed from C?; footprint (none) -> Capacitor_THT:C_Axial_L3.8mm_D2.6mm_P7.50mm_Horizontal
- R2, R3, R4, R5, R6: renamed from R?; footprint (none) -> Resistor_SMD:R_1206_3216Metric
- U3: renamed from U?; footprint (none) -> Package_DIP:DIP-8-16_W7.62mm
- gave numbers to parts that had none: 1
Changed lines of the file:
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@@
   (symbol (lib_id "power:GND") (at 160.02 105.41 270) (unit 1)
     (in_bom yes) (on_board yes)
-    (property "Reference" "#PWR?" (id 0) (at 153.67 105.41 0)
+    (property "Reference" "#PWR0115" (id 0) (at 153.67 105.41 0)
       (effects (font (size 1.27 1.27)) hide)
     )
@@
   (symbol (lib_id "Device:R") (at 69.85 82.55 0) (unit 1)
     (in_bom yes) (on_board yes) (fields_autoplaced)
-    (property "Reference" "R?" (id 0) (at 71.628 81.7153 0)
+    (property "Reference" "R2" (id 0) (at 71.628 81.7153 0)
       (effects (font (size 1.27 1.27)) (justify left))
     )
@@
       (effects (font (size 1.27 1.27)) (justify left))
     )
-    (property "Footprint" "" (id 2) (at 68.072 82.55 90)
+    (property "Footprint" "Resistor_SMD:R_1206_3216Metric" (id 2) (at 68.072 82.55 90)
       (effects (font (size 1.27 1.27)) hide)
     )
@@
   (symbol (lib_id "Amplifier_Operational:LM741") (at 107.95 91.44 0) (unit 1)
     (in_bom yes) (on_board yes)
-    (property "Reference" "U?" (id 0) (at 116.9254 87.6133 0))
+    (property "Reference" "U3" (id 0) (at 116.9254 87.6133 0))
     (property "Value" "LM741" (id 1) (at 110.49 87.63 0))
-    (property "Footprint" "" (id 2) (at 109.22 90.17 0)
+    (property "Footprint" "Package_DIP:DIP-8-16_W7.62mm" (id 2) (at 109.22 90.17 0)
       (effects (font (size 1.27 1.27)) hide)
     )
@@
   (symbol (lib_id "Device:C") (at 195.58 81.28 90) (unit 1)
     (in_bom yes) (on_board yes) (fields_autoplaced)
-    (property "Reference" "C?" (id 0) (at 195.58 75.4212 90))
+    (property "Reference" "C2" (id 0) (at 195.58 75.4212 90))
     (property "Value" "2u" (id 1) (at 195.58 77.9581 90))
-    (property "Footprint" "" (id 2) (at 199.39 80.3148 0)
+    (property "Footprint" "Capacitor_THT:C_Axial_L3.8mm_D2.6mm_P7.50mm_Horizontal" (id 2) (at 199.39 80.3148 0)
       (effects (font (size 1.27 1.27)) hide)
     )
@@
   (symbol (lib_id "Device:R") (at 176.53 81.28 90) (unit 1)
     (in_bom yes) (on_board yes) (fields_autoplaced)
-    (property "Reference" "R?" (id 0) (at 176.53 76.5642 90))
+    (property "Reference" "R6" (id 0) (at 176.53 76.5642 90))
     (property "Value" "100k" (id 1) (at 176.53 79.1011 90))
-    (property "Footprint" "" (id 2) (at 176.53 83.058 90)
+    (property "Footprint" "Resistor_SMD:R_1206_3216Metric" (id 2) (at 176.53 83.058 90)
       (effects (font (size 1.27 1.27)) hide)
     )
@@
   (symbol (lib_id "Device:R") (at 161.29 81.28 90) (unit 1)
     (in_bom yes) (on_board yes) (fields_autoplaced)
-    (property "Reference" "R?" (id 0) (at 161.29 76.5642 90))
+    (property "Reference" "R5" (id 0) (at 161.29 76.5642 90))
     (property "Value" "1k" (id 1) (at 161.29 79.1011 90))
-    (property "Footprint" "" (id 2) (at 161.29 83.058 90)
+    (property "Footprint" "Resistor_SMD:R_1206_3216Metric" (id 2) (at 161.29 83.058 90)
       (effects (font (size 1.27 1.27)) hide)
     )
@@
   (symbol (lib_id "power:+5V") (at 180.34 95.25 0) (unit 1)
     (in_bom yes) (on_board yes) (fields_autoplaced)
-    (property "Reference" "#PWR?" (id 0) (at 180.34 99.06 0)
+    (property "Reference" "#PWR0113" (id 0) (at 180.34 99.06 0)
       (effects (font (size 1.27 1.27)) hide)
     )
@@
   (symbol (lib_id "Device:R") (at 69.85 95.25 0) (unit 1)
     (in_bom yes) (on_board yes) (fields_autoplaced)
-    (property "Reference" "R?" (id 0) (at 71.628 94.4153 0)
+    (property "Reference" "R3" (id 0) (at 71.628 94.4153 0)
       (effects (font (size 1.27 1.27)) (justify left))
     )
@@
       (effects (font (size 1.27 1.27)) (justify left))
     )
-    (property "Footprint" "" (id 2) (at 68.072 95.25 90)
+    (property "Footprint" "Resistor_SMD:R_1206_3216Metric" (id 2) (at 68.072 95.25 90)
       (effects (font (size 1.27 1.27)) hide)
     )
@@
   (symbol (lib_id "Timer:NE555P") (at 180.34 105.41 0) (unit 1)
     (in_bom yes) (on_board yes) (fields_autoplaced)
-    (property "Reference" "U?" (id 0) (at 182.3594 94.0902 0)
+    (property "Reference" "U4" (id 0) (at 182.3594 94.0902 0)
       (effects (font (size 1.27 1.27)) (justify left))
     )
@@
   (symbol (lib_id "power:GND") (at 69.85 101.6 0) (unit 1)
     (in_bom yes) (on_board yes) (fields_autoplaced)
-    (property "Reference" "#PWR?" (id 0) (at 69.85 107.95 0)
+    (property "Reference" "#PWR0109" (id 0) (at 69.85 107.95 0)
       (effects (font (size 1.27 1.27)) hide)
     )
@@
   (symbol (lib_id "power:GND") (at 180.34 115.57 0) (unit 1)
     (in_bom yes) (on_board yes) (fields_autoplaced)
-    (property "Reference" "#PWR?" (id 0) (at 180.34 121.92 0)
+    (property "Reference" "#PWR0114" (id 0) (at 180.34 121.92 0)
       (effects (font (size 1.27 1.27)) hide)
     )
@@
   (symbol (lib_id "Device:R") (at 78.74 74.93 90) (unit 1)
     (in_bom yes) (on_board yes)
-    (property "Reference" "R?" (id 0) (at 78.74 77.47 90))
+    (property "Reference" "R4" (id 0) (at 78.74 77.47 90))
     (property "Value" "1" (id 1) (at 78.74 72.7511 90))
-    (property "Footprint" "" (id 2) (at 78.74 76.708 90)
+    (property "Footprint" "Resistor_SMD:R_1206_3216Metric" (id 2) (at 78.74 76.708 90)
       (effects (font (size 1.27 1.27)) hide)
     )
@@
   (symbol (lib_id "power:GND") (at 213.36 82.55 0) (unit 1)
     (in_bom yes) (on_board yes) (fields_autoplaced)
-    (property "Reference" "#PWR?" (id 0) (at 213.36 88.9 0)
+    (property "Reference" "#PWR0112" (id 0) (at 213.36 88.9 0)
       (effects (font (size 1.27 1.27)) hide)
     )
@@
   (symbol (lib_id "power:GND") (at 105.41 99.06 0) (unit 1)
     (in_bom yes) (on_board yes) (fields_autoplaced)
-    (property "Reference" "#PWR?" (id 0) (at 105.41 105.41 0)
+    (property "Reference" "#PWR0110" (id 0) (at 105.41 105.41 0)
       (effects (font (size 1.27 1.27)) hide)
     )
@@
   (symbol (lib_id "Device:C") (at 163.83 105.41 270) (unit 1)
     (in_bom yes) (on_board yes)
-    (property "Reference" "C?" (id 0) (at 161.29 104.14 90))
+    (property "Reference" "C1" (id 0) (at 161.29 104.14 90))
     (property "Value" "100n" (id 1) (at 163.83 102.0881 90))
-    (property "Footprint" "" (id 2) (at 160.02 106.3752 0)
+    (property "Footprint" "Capacitor_SMD:CP_Elec_3x5.3" (id 2) (at 160.02 106.3752 0)
       (effects (font (size 1.27 1.27)) hide)
     )
@@
   (symbol (lib_id "power:+5V") (at 105.41 83.82 0) (unit 1)
     (in_bom yes) (on_board yes) (fields_autoplaced)
-    (property "Reference" "#PWR?" (id 0) (at 105.41 87.63 0)
-      (effects (font (size 1.27 1.27)) hide)
-    )
+    (property "Reference" "#PWR0111" (id 0) (at 105.41 87.63 0)
+      (effects (font (size 1.27 1.27)) hide)
+    )
